Commit message: added camera to urdf

File: urdf/omni_bot.urdf (robot description, URDF)
Before this commit: robot omni_bot, 5 links, 4 joints
Links:
- added link camera_link, mass 0.1; visual box size=0.03 0.03 0.03
- added link camera_link_optical
Joints:
- added joint camera_joint: type fixed, parent base_footprint, child camera_link, origin xyz=0 0 0.3 rpy=0 0 0
- added joint camera_optical_joint: type fixed, parent camera_link, child camera_link_optical, origin xyz=0 0 0 rpy=-1.5708 0 -1.5708

Commit message: fixed movement by changing mass+friction

File: urdf/omni_bot.urdf (robot description, URDF)
Before this commit: robot omni_bot, 7 links, 6 joints
Links:
- link base_footprint: mass 5.0 -> 2.0
- link wheel_back_left: mass 0.3 -> 0.1
- link wheel_back_right: mass 0.3 -> 0.1
- link wheel_front_left: mass 0.3 -> 0.1
- link wheel_front_right: mass 0.3 -> 0.1
